File: displayboard/Displayboard.kicad_pcb (KiCad board)
At the start: 2 copper layers, 106 x 80 mm, 27 parts, among them IC401 PCAL6416AHF, Q501 NPN, SW401 Button 1, SW402 Button 2, SW403 Button 3, SW404 Button 4, X501 Touch, X502 Display, X503 Mainboard

Commit message: Prepare Release 1.0.0
Parts:
- R501: moved to F.Cu
- X502: footprint Connector_FFC-FPC:TE_1-84952-8_1x18-1MP_P1.0mm_Horizontal -> Molex_Kampi:5051101892
- moved R501 45.7 mm to (244.8, 110.8)
- moved X502 26.4 mm to (218.5, 112.0)
- moved X501 18.0 mm to (199.0, 94.4)
- moved R502 17.8 mm to (217.4, 121.5), turned to 0 degrees
- moved Q501 10.3 mm to (213.4, 121.5), turned to 0 degrees
- moved R503 5.80 mm to (210.3, 121.5), turned to -90 degrees
- moved R504 2.19 mm to (212.0, 124.2)
Connections:
- X501 pad MP: (no net) -> GND
- X502 pad MP: (no net) -> GND
Routing:
- net /Project Architecture/Connectors/SPI-MISO: track 64.7 -> 16.0 mm, vias 2 -> 1
- net /Project Architecture/Connectors/~{Display-CS}: track 66.3 -> 40.4 mm
- net /Project Architecture/Connectors/SPI-SCLK: track 63.2 -> 37.7 mm
- net /Project Architecture/Connectors/SPI-MOSI: track 67.8 -> 42.5 mm
- net /Project Architecture/Connectors/Display-DC: track 64.8 -> 39.9 mm
- net /Project Architecture/Connectors/~{Display-Reset}: track 61.7 -> 37.2 mm
- net Net-(X502-Pin_12): track 2.69 -> 25.2 mm, vias 0 -> 1
- net /Project Architecture/Connectors/I2C-SDA: track 85.5 -> 68.7 mm
- net /Project Architecture/Connectors/I2C-SCL: track 85.9 -> 69.2 mm
- net /Project Architecture/Connectors/~{Touch-IRQ}: track 60.4 -> 44.6 mm
- net /Project Architecture/Connectors/~{Touch-Reset}: track 59.5 -> 43.7 mm
- net Net-(X502-Pin_5): track 5.59 -> 10.9 mm
- net /Project Architecture/Connectors/Display-Backlight: track 57.5 -> 56.0 mm
- net +3V3: track 11.2 -> 9.78 mm
- net Net-(IC401-P0_1): track 39.1 -> 38.3 mm
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Other:
- outline, holes or cut-outs redrawn

Commit message: Update outputs (release)
Other:
- board text added: "0.035mm (1.00oz)"
- board text added: "1.0mm"
- board text added: "Total thickness: 1.09mm"
- board text removed: "0.035mm (1oz)"
- board text removed: "1.51mm"
- board text removed: "Total thickness: 1.6mm"
